File: Split_keyboard_analog_pad/Split_keyboard_analog_pad.kicad_pcb (KiCad board)
At the start: 2 copper layers, 313.3 x 128.7 mm, 160 parts, among them J1 Conn_01x05_Pin, J2 Conn_01x05_Pin, J3 Conn_01x08_Pin, J4 Conn_01x08_Pin, M2 MountingHole_2.2mm_M2, U1 nice_nano, U2 nice_nano

Commit message: remove LED definition
Parts:
- added D1: WS2812B, LED_SMD:LED_WS2812B_PLCC4_5.0x5.0mm_P3.2mm, F.Cu at (84.0, -88.5)
- added D2: WS2812B, LED_SMD:LED_WS2812B_PLCC4_5.0x5.0mm_P3.2mm, F.Cu at (92.5, -88.5)
- renumbered BATTERY to J5, BATTERY to J6
Connections:
- U1 pad 15: unconnected-(U1-P1.11-Pad15) -> /LED_CTRL
- U1 pad 21: unconnected-(U1-VCC-Pad21) -> /VCC_L
Routing:
- net /VCC_L: track 0.00 -> 113.7 mm, vias 0 -> 1
- net /GND_L: track 35.5 -> 144.5 mm, vias 1 -> 4
- net /LED_CTRL: track 0.00 -> 107.7 mm, vias 0 -> 2
- net Net-(D1-DOUT): track 0.00 -> 14.8 mm
- net /RL0: track 172.4 -> 174.2 mm
- net /RL4: track 201.5 -> 200.3 mm
- net /RL3: track 208.6 -> 209.2 mm
Other:
- board text added: "nice!nano"
